File: clocks.sch (KiCad schematic (older format))
At the start: 18 parts, among them J4 UPDI TTL, U10 ATtiny1614-SS, U11 ACDA02-41SGWA-F01, U12 AS1115-BSST, U7 TPS7A0533PDBVR, U8 74HC04, U9 Si5351A-B-GT, Y1 25MHZ 8PF

Commit message: removed rescue and cache from .gitignore
Parts:
- U11: symbol sbc_z80-rescue:ACDA02-41SGWA-F01-Display_Character -> z180_motherboard-rescue:ACDA02-41SGWA-F01-Display_Character-sbc_z80-rescue
- U7: symbol sbc_z80-rescue:TPS7A0533PDBVR-Regulator_Linear -> z180_motherboard-rescue:TPS7A0533PDBVR-Regulator_Linear-sbc_z80-rescue
Connections:
- net labels added: CLK_50Mhz
- net labels removed: CLK_100Mhz
Changed lines of the file:
@@
 	8845 1305 8845 1080
 $Comp
-L sbc_z80-rescue:TPS7A0533PDBVR-Regulator_Linear U7
+L z180_motherboard-rescue:TPS7A0533PDBVR-Regulator_Linear-sbc_z80-rescue U7
 U 1 1 5D35A913
 P 1980 1045
@@
 $EndComp
 Text HLabel 9445 1080 2    50   Output ~ 0
-CLK_100Mhz
+CLK_50Mhz
 Text HLabel 9440 1925 2    50   Output ~ 0
 CLK_7_3728_Mhz
 Text HLabel 9440 1505 2    50   Output ~ 0
 CLK_10_Mhz
-Wire Bus Line
-	3595 3415 3595 4690
-Wire Bus Line
-	4225 3580 4225 4640
-Wire Bus Line
-	5945 3580 5945 4640
 Wire Wire Line
 	2635 3330 2635 3285
@@
 $EndComp
 $Comp
-L sbc_z80-rescue:ACDA02-41SGWA-F01-Display_Character U?
+L z180_motherboard-rescue:ACDA02-41SGWA-F01-Display_Character-sbc_z80-rescue U?
 U 1 1 5F4897F6
 P 5085 4185
@@
 	1    0    0    -1
 $EndComp
+Wire Bus Line
+	5945 3580 5945 4640
+Wire Bus Line
+	4225 3580 4225 4640
+Wire Bus Line
+	3595 3415 3595 4690
 $EndSCHEMATC
